File: hardware/rain/rev_a/rain.brd (EAGLE design)
At the start: 25.4 x 21 mm, 23 parts, among them J1 SQUALL_HEADER, U1 ADXL362, U2 LPS331AP, U3 ML8511, U4 SI1141, U5 SI7021, U6 SI1147, U7 MPU-9250

Commit message: rain getting close
Parts:
- removed C11, C13: 0.1uF, passives:0402_CAP
- removed C12: CAP_POL0603, passives:CAP0603
- removed U5: SI7021, chips:DFN-6/3MM
- removed U6: SI1147, chips:QFN-10/2MM
- removed U7: MPU-9250, chips:QFN-24/3MM
- added C1: 10nF, passives:0402_CAP
- added C10: 22uF, passives:CAP0603
- added C8: 0.1uF, passives:0402_CAP
- added C9: 10uF, passives:0402_CAP
- added D4: DIODE, passives:0402_DIODE
- added J2: (no value), pinhead:2X02
- added LOGO1: UMICH_SOLID_TINY, logos:UMICH_SOLID_50MIL
- added M1: 308-100, motor:308-100
- added Q1: ROHM-NPN-2SC5662, fets:VMT3
- added R4, R5: 10k, passives:0402_RES
- C3: value 10nF -> 0.1uF
- C6: value 10uF -> 0.1uF
- R2: value 10k -> 33
- R3: value 10k -> 1k
- U1: value ADXL362 -> LPS331AP; device chips:TFLGA-16/3.3MMX3.1MM -> chips:HCLGA-16/3MM
- U2: value LPS331AP -> MPU-9250; device chips:HCLGA-16/3MM -> chips:QFN-24/3MM
- U3: value ML8511 -> SI1147; device chips:TQFN-12/4MM -> chips:QFN-10/2MM
- U4: value SI1141 -> SI7021; device chips:QFN-10/2MM -> chips:DFN-6/3MM
- moved U3 31.0 mm to (8.13, 7.49)
- moved U4 25.5 mm to (12.7, 1.91)
- moved R3 23.0 mm to (13.3, 18.9)
- moved U1 17.2 mm to (14.6, 14.5), turned to 90 degrees
- moved R2 15.2 mm to (9.65, 12.7), turned to 270 degrees
- moved D1 14.0 mm to (6.35, 19.1), turned to 180 degrees
- moved D3 14.0 mm to (20.3, 19.1), turned to 180 degrees
- moved C7 12.6 mm to (5.97, 6.73), turned to 270 degrees
- moved C5 11.9 mm to (19.4, 8.13), turned to 0 degrees
- moved R1 7.73 mm to (3.17, 18.9), turned to 270 degrees
- moved C2 7.30 mm to (13.1, 11.9)
- moved U2 7.22 mm to (16.4, 9.14)
- moved C6 5.46 mm to (9.65, 17.8), turned to 180 degrees
- moved C3 5.38 mm to (11.7, 15.2)
- moved D2 0.51 mm to (6.35, 4.57), turned to 180 degrees
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Connections:
- removed net UV_ADC: U3.8
- removed net UV_EN: U3.4
- new net A7: J1.B5, J2.2
- new net MOTOR_CTRL: J1.A2, J2.4, R3.2
- new net N$5: Q1.1, R3.1
- net !ACCEL_CS: now also J1.B7, U2.22; no longer U7.22
- net !PRESSURE_CS: now also J1.A4, U1.8; no longer U2.8
- net ACCEL_INT: now also J1.B9, U2.12; no longer U7.12
- net GND: now also C1.2, C10.NEG, C8.2, C9.2, J1.A10, J1.A9, J2.1, Q1.2, U1.10, U1.12, U1.13, U1.16, U1.5, U2.11, U2.18, U2.20, U3.8, U4.2; no longer C11.2, C12.NEG, C13.2, C6.2, U2.10, U2.12, U2.13, U2.16, U2.5, U5.2, U6.8, U7.11, U7.18, U7.20
- net LIGHT_INT: now also J1.A8, U3.4; no longer U6.4
- net MISO: now also U1.7, U2.9; no longer U2.7, U7.9
- net MOSI: now also U1.6, U2.24; no longer U2.6, U7.24
- net N$1: now also C6.1, D4.CATHODE, M1.POS, R2.1; no longer U4.3, U4.6, U4.7
- net N$2: now also C6.2, D4.ANODE, M1.NEG, Q1.3; no longer J1.A10, J1.A9
- net N$3: now also U2.10; no longer U7.10
- net N$4: now also U3.9; no longer U6.9
- net N$6: now also U3.6; no longer U6.6
- net N$7: now also U3.7; no longer U6.7
- net N$8: now also C10.POS; no longer C12.POS
- net PRESSURE_INT: now also J1.A6, U1.11; no longer U2.11
- net SCL: now also R5.1, U3.2, U4.6; no longer R3.1, U5.6, U6.2
- net SCLK: now also U1.4, U2.23; no longer U2.4, U7.23
- net SDA: now also R4.1, U3.1, U4.1; no longer R2.1, U5.1, U6.1
- net VCC: now also C1.1, C8.1, C9.1, J2.3, R4.2, R5.2, U1.1, U1.14, U1.15, U2.13, U2.8, U3.3, U4.5; no longer C11.1, C13.1, C6.1, R3.2, U2.14, U2.15, U5.5, U6.3, U7.1, U7.13, U7.8
Routing:
- net VCC: track 0.00 -> 71.2 mm, vias 0 -> 4
- net N$8: track 0.00 -> 33.9 mm
- net GND: track 0.00 -> 31.6 mm, vias 0 -> 13
- net N$7: track 0.00 -> 23.3 mm
- net MOTOR_CTRL: track 0.00 -> 20.6 mm, vias 0 -> 1
- net LIGHT_INT: track 0.00 -> 13.6 mm, vias 0 -> 1
- net !PRESSURE_CS: track 0.00 -> 13.4 mm, vias 0 -> 1
- net PRESSURE_INT: track 0.00 -> 11.7 mm, vias 0 -> 1
- net N$4: track 0.00 -> 11.4 mm
- net N$2: track 0.00 -> 7.18 mm, vias 0 -> 1
- net !ACCEL_CS: track 0.00 -> 6.51 mm, vias 0 -> 1
- net N$1: track 0.00 -> 6.01 mm
- net MOSI: track 11.5 -> 17.4 mm, vias 1 -> 3
- net A7: track 0.00 -> 5.42 mm
- net ACCEL_INT: track 0.00 -> 4.64 mm, vias 0 -> 1
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- added copper zone on layer 16, net GND
Other:
- board text added: "A"
- board text added: "A7"
- board text added: "Brad Campbell"
- board text added: "GND"
- board text added: "P22"
- board text added: "VCC"
- board text added: "X"
- board text added: "Y"
- board text added: "Z"
