File: hardware/rain/rev_a/rain.sch (EAGLE design)
At the start: 23 parts, among them J1 SQUALL_HEADER, U1 ADXL362, U2 LPS331AP, U3 ML8511, U4 SI1141, U5 SI7021, U6 SI1147, U7 MPU-9250

Commit message: rain getting close
Parts:
- removed C11, C13: 0.1uF, passives:CAPACITOR
- removed C12: CAP_POL0603, passives:CAP_POL0603
- removed U5: SI7021, chips:SI7021
- removed U6: SI1147, chips:SI1147
- removed U7: MPU-9250, chips:MPU-9250
- added C1: 10nF, passives:CAPACITOR
- added C10: 22uF, passives:CAP_POL0603
- added C8: 0.1uF, passives:CAPACITOR
- added C9: 10uF, passives:CAPACITOR
- added D4: DIODE, passives:DIODE
- added J2: (no value), pinhead:PINHD-2X2
- added LOGO1: UMICH_SOLID_TINY, logos:UMICH_SOLID_TINY
- added M1: 308-100, motor:308-100
- added Q1: ROHM-NPN-2SC5662, fets:ROHM-NPN-2SC5662
- added R4, R5: 10k, passives:RESISTOR0402_RES
- C3: value 10nF -> 0.1uF
- C6: value 10uF -> 0.1uF
- R2: value 10k -> 33
- R3: value 10k -> 1k
- U1: value ADXL362 -> LPS331AP; device chips:ADXL362 -> chips:LPS331AP
- U2: value LPS331AP -> MPU-9250; device chips:LPS331AP -> chips:MPU-9250
- U3: value ML8511 -> SI1147; device chips:ML8511 -> chips:SI1147
- U4: value SI1141 -> SI7021; device chips:SI1141 -> chips:SI7021
Connections:
- removed net UV_ADC: U3.OUT
- removed net UV_EN: U3.EN
- new net A7: J1.A7, J2.2
- new net MOTOR_CTRL: J1.P22, J2.4, R3.2
- new net N$5: Q1.BASE, R3.1
- net !ACCEL_CS: now also J1.A6, U2.!CS; no longer U7.!CS
- net !PRESSURE_CS: now also J1.P23, U1.!CS; no longer U2.!CS
- net ACCEL_INT: now also J1.A5, U2.INT; no longer U7.INT
- net GND: now also C1.2, C10.ANODE, C8.2, C9.2, J1.GND, J2.1, Q1.EMITTER, U1.GND, U2.FSYNC, U3.GND, U4.GND; no longer C11.2, C12.ANODE, C13.2, C6.2, U5.GND, U6.GND, U7.FSYNC, U7.GND
- net LIGHT_INT: now also J1.P25, U3.INT; no longer U6.INT
- net MISO: now also U1.SA0/MISO, U2.AD0/MISO; no longer U2.SA0/MISO, U7.AD0/MISO
- net MOSI: now also U1.SDA/MOSI; no longer U7.SDA/MOSI
- net N$1: now also C6.1, D4.CATHODE, M1.POS, R2.1; no longer U4.VCC
- net N$2: now also C6.2, D4.ANODE, M1.NEG, Q1.COLLECTOR; no longer J1.GND
- net N$3: now also U2.REGOUT; no longer U7.REGOUT
- net N$4: now also U3.LED1; no longer U6.LED1
- net N$6: now also U3.LED2; no longer U6.LED2
- net N$7: now also U3.LED3; no longer U6.LED3
- net N$8: now also C10.CATHODE; no longer C12.CATHODE
- net PRESSURE_INT: now also J1.P24, U1.INT1; no longer U2.INT1
- net SCL: now also R5.1, U3.SCL, U4.SCL; no longer R3.1, U5.SCL, U6.SCL
- net SCLK: now also U1.SCLK; no longer U7.SCLK
- net SDA: now also R4.1, U3.SDA, U4.SDA; no longer R2.1, U5.SDA, U6.SDA
- net VCC: now also C1.1, C8.1, C9.1, J2.3, R4.2, R5.2, U1.VCC, U1.VCCA, U1.VDDIO, U2.VDD, U3.VDD, U4.VCC; no longer C11.1, C13.1, C6.1, R3.2, U2.VCC, U2.VCCA, U5.VCC, U6.VDD, U7.VDD, U7.VDDIO
Other:
- note added: "9-DOF Accelerometer"
- note added: "Light/UV/Proximity Sensor"
- note added: "Pin Header"
- note added: "Pressure Sensor"
- note added: "Squall Header"
- note added: "Temperature/Humidity Sensor"
- note added: "Vibration Motor"
- moved on the sheet: C2, C3, C4, C5, C6, C7, D1, D2, D3, R1, R2, R3

Commit message: rain pretty much done
needs a name
Parts:
- C1: DIGIKEY (none) -> 490-1312-1-ND
- C10: DIGIKEY (none) -> 511-1493-1-ND
- C2, C3, C4, C5, C6, C7, C8: DIGIKEY (none) -> 490-1318-1-ND
- C9: DIGIKEY (none) -> 445-8919-1-ND
- J2: DIGIKEY (none) -> 609-3201-ND
- R1: DIGIKEY (none) -> RHM30CECT-ND
- R2: DIGIKEY (none) -> RHM33CECT-ND
- R3: DIGIKEY (none) -> RHM1.0KCECT-ND
- R4, R5: DIGIKEY (none) -> RHM10.0KCDCT-ND
