File: hardware/squall/rev_a/squall.sch (EAGLE design)
At the start: 38 parts, among them J1 HIROSE-DF40C-10DP-0.4V, J2 HIROSE-DF40C-10DP-0.4V, J3 MICRO_USB_B_JST_MC5BR3-M404-4S, J4 TC2030-JLINK-NL, U1 NRF51822QF, U2 FT232RQ, X1 16MHz, X2 ABS05-32.768KHZ-9-T

Commit message: updated a digikey part num
Parts:
- C1: DIGIKEY 490-5419-1-ND -> 490-6269-1-ND
Changed lines of the file:
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@@
 <part name="FRAME2" library="frames" deviceset="LETTER_L" device=""/>
 <part name="C1" library="passives" deviceset="CAPACITOR" device="" value="0.8pF">
-<attribute name="DIGIKEY" value="490-5419-1-ND"/>
+<attribute name="DIGIKEY" value="490-6269-1-ND"/>
 </part>
 <part name="GND10" library="supply1" deviceset="GND" device=""/>

Commit message: fixes: battery location and ftdi
- rotated battery clip to hopefully not conflict with mounting holes
- connected test on FTDI to gnd
Connections:
- removed net P07: U1.P07
- removed net P12: U1.P12
- removed net P21: U1.P21
- net GND: now also U2.GND, U2.GND@1, U2.GND@2, U2.TEST
- net SCL: now also U1.P07
Changed lines of the file:
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@@
 <part name="GND15" library="supply1" deviceset="GND" device=""/>
 <part name="P+1" library="supply1" deviceset="VCC" device=""/>
+<part name="GND3" library="supply1" deviceset="GND" device=""/>
 </parts>
 <sheets>
@@
 </segment>
 </net>
-<net name="P12" class="0">
-<segment>
-<pinref part="U1" gate="G$1" pin="P12"/>
-<wire x1="55.88" y1="76.2" x2="53.34" y2="76.2" width="0.1524" layer="91"/>
-<label x="53.34" y="76.2" size="1.27" layer="95" rot="R180" xref="yes"/>
-</segment>
-</net>
 <net name="PROG_RX" class="0">
 <segment>
@@
 </segment>
 </net>
-<net name="P07" class="0">
+<net name="P23" class="0">
+<segment>
+<pinref part="U1" gate="G$1" pin="P23"/>
+<wire x1="101.6" y1="96.52" x2="104.14" y2="96.52" width="0.1524" layer="91"/>
+<label x="104.14" y="96.52" size="1.27" layer="95" xref="yes"/>
+</segment>
+<segment>
+<pinref part="J1" gate="G$1" pin="4"/>
+<wire x1="185.42" y1="139.7" x2="177.8" y2="139.7" width="0.1524" layer="91"/>
+<label x="185.42" y="139.7" size="1.27" layer="95" xref="yes"/>
+</segment>
+</net>
+<net name="P22" class="0">
+<segment>
+<pinref part="U1" gate="G$1" pin="P22"/>
+<wire x1="101.6" y1="99.06" x2="104.14" y2="99.06" width="0.1524" layer="91"/>
+<label x="104.14" y="99.06" size="1.27" layer="95" xref="yes"/>
+</segment>
+<segment>
+<pinref part="J1" gate="G$1" pin="2"/>
+<wire x1="185.42" y1="142.24" x2="177.8" y2="142.24" width="0.1524" layer="91"/>
+<label x="185.42" y="142.24" size="1.27" layer="95" xref="yes"/>
+</segment>
+</net>
+<net name="BTLDR_CTRL" class="0">
+<segment>
+<pinref part="U1" gate="G$1" pin="P03/AIN4"/>
+<wire x1="55.88" y1="101.6" x2="53.34" y2="101.6" width="0.1524" layer="91"/>
+<label x="53.34" y="101.6" size="1.27" layer="95" rot="R180" xref="yes"/>
+</segment>
+</net>
+<net name="P25" class="0">
+<segment>
+<pinref part="U1" gate="G$1" pin="P25"/>
+<wire x1="101.6" y1="88.9" x2="104.14" y2="88.9" width="0.1524" layer="91"/>
+<label x="104.14" y="88.9" size="1.27" layer="95" xref="yes"/>
+</segment>
+<segment>
+<pinref part="J1" gate="G$1" pin="8"/>
+<wire x1="177.8" y1="134.62" x2="185.42" y2="134.62" width="0.1524" layer="91"/>
+<label x="185.42" y="134.62" size="1.27" layer="95" xref="yes"/>
+</segment>
+</net>
+<net name="N$8" class="0">
+<segment>
+<pinref part="R1" gate="G$1" pin="2"/>
+<pinref part="S1" gate="G$1" pin="P$2"/>
+<wire x1="43.18" y1="45.72" x2="43.18" y2="48.26" width="0.1524" layer="91"/>
+</segment>
+</net>
+<net name="SCL" class="0">
+<segment>
+<pinref part="J2" gate="G$1" pin="3"/>
+<wire x1="210.82" y1="139.7" x2="205.74" y2="139.7" width="0.1524" layer="91"/>
+<label x="205.74" y="139.7" size="1.27" layer="95" rot="R180" xref="yes"/>
+</segment>
 <segment>
 <pinref part="U1" gate="G$1" pin="P07"/>
 <wire x1="55.88" y1="91.44" x2="53.34" y2="91.44" width="0.1524" layer="91"/>
 <label x="53.34" y="91.44" size="1.27" layer="95" rot="R180" xref="yes"/>
-</segment>
-</net>
-<net name="P23" class="0">
-<segment>
-<pinref part="U1" gate="G$1" pin="P23"/>
-<wire x1="101.6" y1="96.52" x2="104.14" y2="96.52" width="0.1524" layer="91"/>
-<label x="104.14" y="96.52" size="1.27" layer="95" xref="yes"/>
-</segment>
-<segment>
-<pinref part="J1" gate="G$1" pin="4"/>
-<wire x1="185.42" y1="139.7" x2="177.8" y2="139.7" width="0.1524" layer="91"/>
-<label x="185.42" y="139.7" size="1.27" layer="95" xref="yes"/>
-</segment>
-</net>
-<net name="P22" class="0">
-<segment>
-<pinref part="U1" gate="G$1" pin="P22"/>
-<wire x1="101.6" y1="99.06" x2="104.14" y2="99.06" width="0.1524" layer="91"/>
-<label x="104.14" y="99.06" size="1.27" layer="95" xref="yes"/>
-</segment>
-<segment>
-<pinref part="J1" gate="G$1" pin="2"/>
-<wire x1="185.42" y1="142.24" x2="177.8" y2="142.24" width="0.1524" layer="91"/>
-<label x="185.42" y="142.24" size="1.27" layer="95" xref="yes"/>
-</segment>
-</net>
-<net name="P21" class="0">
-<segment>
-<pinref part="U1" gate="G$1" pin="P21"/>
-<wire x1="101.6" y1="101.6" x2="104.14" y2="101.6" width="0.1524" layer="91"/>
-<label x="104.14" y="101.6" size="1.27" layer="95" xref="yes"/>
-</segment>
-</net>
-<net name="BTLDR_CTRL" class="0">
-<segment>
-<pinref part="U1" gate="G$1" pin="P03/AIN4"/>
-<wire x1="55.88" y1="101.6" x2="53.34" y2="101.6" width="0.1524" layer="91"/>
-<label x="53.34" y="101.6" size="1.27" layer="95" rot="R180" xref="yes"/>
-</segment>
-</net>
-<net name="P25" class="0">
-<segment>
-<pinref part="U1" gate="G$1" pin="P25"/>
-<wire x1="101.6" y1="88.9" x2="104.14" y2="88.9" width="0.1524" layer="91"/>
-<label x="104.14" y="88.9" size="1.27" layer="95" xref="yes"/>
-</segment>
-<segment>
-<pinref part="J1" gate="G$1" pin="8"/>
-<wire x1="177.8" y1="134.62" x2="185.42" y2="134.62" width="0.1524" layer="91"/>
-<label x="185.42" y="134.62" size="1.27" layer="95" xref="yes"/>
-</segment>
-</net>
-<net name="N$8" class="0">
-<segment>
-<pinref part="R1" gate="G$1" pin="2"/>
-<pinref part="S1" gate="G$1" pin="P$2"/>
-<wire x1="43.18" y1="45.72" x2="43.18" y2="48.26" width="0.1524" layer="91"/>
-</segment>
-</net>
-<net name="SCL" class="0">
-<segment>
-<pinref part="J2" gate="G$1" pin="3"/>
-<wire x1="210.82" y1="139.7" x2="205.74" y2="139.7" width="0.1524" layer="91"/>
-<label x="205.74" y="139.7" size="1.27" layer="95" rot="R180" xref="yes"/>
 </segment>
 </net>
@@
 <attribute name="MOUSER" x="81.28" y="160.02" size="1.27" layer="96" display="off"/>
 </instance>
+<instance part="GND3" gate="1" x="170.18" y="35.56"/>
 </instances>
 <busses>
@@
 <pinref part="GND4" gate="1" pin="GND"/>
 </segment>
-</net>
+<segment>
+<pinref part="U2" gate="1" pin="TEST"/>
+<wire x1="167.64" y1="53.34" x2="170.18" y2="53.34" width="0.1524" layer="91"/>
+<wire x1="170.18" y1="53.34" x2="170.18" y2="48.26" width="0.1524" layer="91"/>
+<pinref part="GND3" gate="1" pin="GND"/>
+<pinref part="U2" gate="1" pin="GND"/>
+<wire x1="170.18" y1="48.26" x2="170.18" y2="45.72" width="0.1524" layer="91"/>
+<wire x1="170.18" y1="45.72" x2="170.18" y2="43.18" width="0.1524" layer="91"/>
+<wire x1="170.18" y1="43.18" x2="170.18" y2="38.1" width="0.1524" layer="91"/>
+<wire x1="167.64" y1="48.26" x2="170.18" y2="48.26" width="0.1524" layer="91"/>
+<junction x="170.18" y="48.26"/>
+<pinref part="U2" gate="1" pin="GND@1"/>
+<wire x1="167.64" y1="45.72" x2="170.18" y2="45.72" width="0.1524" layer="91"/>
+<junction x="170.18" y="45.72"/>
+<pinref part="U2" gate="1" pin="GND@2"/>
+<wire x1="167.64" y1="43.18" x2="170.18" y2="43.18" width="0.1524" layer="91"/>
+<junction x="170.18" y="43.18"/>
+</segment>
+</net>
