File: hardware/squall/rev_a/squall.sch (EAGLE design)
At the start: 38 parts, among them J1 HIROSE-DF40C-10DP-0.4V, J2 HIROSE-DF40C-10DP-0.4V, J3 MICRO_USB_B_JST_MC5BR3-M404-4S, J4 TC2030-JLINK-NL, U1 NRF51822QF, U2 FT232RQ, X1 16MHz, X2 ABS05-32.768KHZ-9-T

Commit message: squall: give all 0.1uF caps the same digikey attr
Parts:
- C10: DIGIKEY 445-4952-1-ND -> 490-1318-6-ND
Changed lines of the file:
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@@
 <parts>
 <part name="C10" library="passives" deviceset="CAPACITOR" device="" value="0.1uF">
-<attribute name="DIGIKEY" value="445-4952-1-ND"/>
+<attribute name="DIGIKEY" value="490-1318-6-ND"/>
 </part>
 <part name="P+6" library="supply1" deviceset="VCC" device=""/>

Commit message: squall: 0.1uF digikey TR -> CT to make scripts happy
Parts:
- C10, C11, C12, C13: DIGIKEY 490-1318-6-ND -> 490-1318-1-ND
Changed lines of the file:
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@@
 <parts>
 <part name="C10" library="passives" deviceset="CAPACITOR" device="" value="0.1uF">
-<attribute name="DIGIKEY" value="490-1318-6-ND"/>
+<attribute name="DIGIKEY" value="490-1318-1-ND"/>
 </part>
 <part name="P+6" library="supply1" deviceset="VCC" device=""/>
@@
 </part>
 <part name="C11" library="passives" deviceset="CAPACITOR" device="" value="0.1uF">
-<attribute name="DIGIKEY" value="490-1318-6-ND"/>
+<attribute name="DIGIKEY" value="490-1318-1-ND"/>
 </part>
 <part name="GND16" library="supply1" deviceset="GND" device=""/>
 <part name="GND17" library="supply1" deviceset="GND" device=""/>
 <part name="C12" library="passives" deviceset="CAPACITOR" device="" value="0.1uF">
-<attribute name="DIGIKEY" value="490-1318-6-ND"/>
+<attribute name="DIGIKEY" value="490-1318-1-ND"/>
 </part>
 <part name="C13" library="passives" deviceset="CAPACITOR" device="" value="0.1uF">
-<attribute name="DIGIKEY" value="490-1318-6-ND"/>
+<attribute name="DIGIKEY" value="490-1318-1-ND"/>
 </part>
 <part name="GND22" library="supply1" deviceset="GND" device=""/>

Commit message: squall: replace obsoleted 1k resistor
Parts:
- R3: DIGIKEY RHM1.0KCECT-ND -> 1276-4376-1-ND
Changed lines of the file:
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@@
 <part name="D1" library="SparkFun-LED" deviceset="LED" device="0603" value="BLUE"/>
 <part name="R3" library="passives" deviceset="RESISTOR" device="" value="1k">
-<attribute name="DIGIKEY" value="RHM1.0KCECT-ND"/>
+<attribute name="DIGIKEY" value="1276-4376-1-ND"/>
 </part>
 <part name="FRAME1" library="frames" deviceset="LETTER_L" device=""/>

Commit message: squall: replace obsoleted 12K resistor
Parts:
- R4: DIGIKEY RHM12.0KCDCT-ND -> 1276-4122-1-ND
Changed lines of the file:
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@@
 <part name="GND20" library="supply1" deviceset="GND" device=""/>
 <part name="R4" library="passives" deviceset="RESISTOR" device="" value="12k">
-<attribute name="DIGIKEY" value="RHM12.0KCDCT-ND"/>
+<attribute name="DIGIKEY" value="1276-4122-1-ND"/>
 </part>
 <part name="GND21" library="supply1" deviceset="GND" device=""/>
