File: hardware/squall/rev_a/squall.sch (EAGLE design)
At the start: 38 parts, among them J1 HIROSE-DF40C-10DP-0.4V, J2 HIROSE-DF40C-10DP-0.4V, J3 MICRO_USB_B_JST_MC5BR3-M404-4S, J4 TC2030-JLINK-NL, U1 NRF51822QF, U2 FT232RQ, X1 16MHz, X2 ABS05-32.768KHZ-9-T

Commit message: squall: update attributes for all parts
Parts:
- C1: DESCRIPTION (none) -> CAP CER 0.8PF 50V C0G/NP0 0402; MANUFACTURER (none) -> Murata; MPN (none) -> GRM1555C1HR80BA01D
- C10, C11, C12, C13: DESCRIPTION (none) -> CAP CER 0.1UF 10V X5R 0402; MANUFACTURER (none) -> Murata; MPN (none) -> GRM155R61A104KA01D
- C14: DESCRIPTION (none) -> 1µF ±10% 6.3V Ceramic Capacitor X7R 0402 (1005 Metric); MANUFACTURER (none) -> Samsung; MPN (none) -> CL05B105KQ5NQNC
- C15: DESCRIPTION (none) -> CAP CER 4.7UF 6.3V X5R 0402; MANUFACTURER (none) -> TDK; MPN (none) -> C1005X5R0J475K050BC
- C2, C3, C4, C5: DESCRIPTION (none) -> CAP CER 12PF 50V C0G/NP0 0402; MANUFACTURER (none) -> Murata; MPN (none) -> GRM1555C1H120GA01D
- C6, C7: DESCRIPTION (none) -> CAP CER 1000PF 50V X7R 0402; MANUFACTURER (none) -> Murata; MPN (none) -> GRM155R71H102KA01D
- C8: DESCRIPTION (none) -> CAP CER 2200PF 25V 10% X7R 0402; MANUFACTURER (none) -> Murata; MPN (none) -> GRM155R71E222KA01D
- C9: DESCRIPTION (none) -> CAP CER 0.047UF 16V X7R 0402; MANUFACTURER (none) -> TDK; MPN (none) -> C1005X7R1C473K050BC
- D2: DESCRIPTION (none) -> DIODE SCHOTTKY 30V 0.1A 0402; MANUFACTURER (none) -> Comchip; MPN (none) -> CDBQR0130L
- L1: DESCRIPTION (none) -> FIXED IND 15NH 320MA 460 MOHM; MANUFACTURER (none) -> Taiyo Yuden; MPN (none) -> HK100515NJ-T
- L2: DESCRIPTION (none) -> FIXED IND 10UH 50MA 900 MOHM SMD; MANUFACTURER (none) -> Murata; MPN (none) -> LQM18FN100M00D
- R1, R2: DESCRIPTION (none) -> RES SMD 150 OHM 1% 1/16W 0402; MANUFACTURER (none) -> Rohm; MPN (none) -> MCR01MRTF1500
- R3: DESCRIPTION (none) -> RES SMD 1K OHM 5% 1/16W 0402; MANUFACTURER (none) -> Samsung; MPN (none) -> RC1005J102CS
- R4: DESCRIPTION (none) -> RES SMD 12K OHM 1% 1/16W 0402; MANUFACTURER (none) -> Samsung; MPN (none) -> RC1005F123CS
- X1: DESCRIPTION (none) -> CRYSTAL 16.0000MHZ 8PF SMD; MANUFACTURER (none) -> TXC; MPN (none) -> 8Y-16.000MAAV-T
